File: hardware/Stuttgart.kicad_pcb (KiCad board)
At the start: 2 copper layers, 70 x 70 mm, 79 parts, among them IC1 NCV1117ST33T3G, IC2 UCC12040DVER, IC3 MCP1700T-3302E_TT, IC4 ISO7763DBQR, IC5 ISO7741DBQR, IC6 MCP3202-CI_SN, IC7 MCP251863T-E_9PX, J1 USB_C_Receptacle_USB2.0_16P, J2 FCR7350B, J3 FCR7350G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

Commit message: Prep for new Isolation concept
Parts:
- moved C21 2.85 mm to (149.9, 105.0)
- moved C18 2.85 mm to (132.2, 105.3)
- moved C20 2.85 mm to (147.9, 105.1)
- moved IC2 2.85 mm to (141.0, 107.8)
- moved TP6 2.85 mm to (149.6, 109.7)
- moved C19 2.85 mm to (134.1, 105.3)
Changed lines of the file:
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@@
 	(footprint "Stuttgart:SOIC127P1030X265-16N"
 		(layer "F.Cu")
-		(at 140.58 105.02)
+		(at 141.025 107.837254)
 		(descr "DVE0016A")
 		(tags "Integrated Circuit")
@@
 	(footprint "Capacitor_SMD:C_0603_1608Metric"
 		(layer "F.Cu")
-		(at 133.68 102.495 90)
+		(at 134.125 105.312254 90)
 		(descr "Capacitor SMD 0603 (1608 Metric), square (rectangular) end terminal, IPC-7351 nominal, (Body size source: IPC-SM-782 page 76, https://www.pcb-3d.com/wordpress/wp-content/uploads/ipc-sm-782a_amendment_1_and_2.pdf)")
 		(tags "capacitor")
@@
 	(footprint "Capacitor_SMD:C_0603_1608Metric"
 		(layer "F.Cu")
-		(at 147.495 102.317747 90)
+		(at 147.94 105.135001 90)
 		(descr "Capacitor SMD 0603 (1608 Metric), square (rectangular) end terminal, IPC-7351 nominal, (Body size source: IPC-SM-782 page 76, https://www.pcb-3d.com/wordpress/wp-content/uploads/ipc-sm-782a_amendment_1_and_2.pdf)")
 		(tags "capacitor")
@@
 	(footprint "Capacitor_SMD:C_0805_2012Metric"
 		(layer "F.Cu")
-		(at 149.42 102.142747 90)
+		(at 149.865 104.960001 90)
 		(descr "Capacitor SMD 0805 (2012 Metric), square (rectangular) end terminal, IPC-7351 nominal, (Body size source: IPC-SM-782 page 76, https://www.pcb-3d.com/wordpress/wp-content/uploads/ipc-sm-782a_amendment_1_and_2.pdf, https://docs.google.com/spreadsheets/d/1BsfQQcO9C6DZCsRaXUlFlo91Tg2WpOkGARC1WS5S8t0/edit?usp=sharing)")
 		(tags "capacitor")
@@
 	(footprint "Capacitor_SMD:C_0805_2012Metric"
 		(layer "F.Cu")
-		(at 131.755 102.52 90)
+		(at 132.2 105.337254 90)
 		(descr "Capacitor SMD 0805 (2012 Metric), square (rectangular) end terminal, IPC-7351 nominal, (Body size source: IPC-SM-782 page 76, https://www.pcb-3d.com/wordpress/wp-content/uploads/ipc-sm-782a_amendment_1_and_2.pdf, https://docs.google.com/spreadsheets/d/1BsfQQcO9C6DZCsRaXUlFlo91Tg2WpOkGARC1WS5S8t0/edit?usp=sharing)")
 		(tags "capacitor")
@@
 	(footprint "TestPoint:TestPoint_Pad_D1.0mm"
 		(layer "F.Cu")
-		(at 149.125 106.867306 -90)
+		(at 149.57 109.68456 -90)
 		(descr "SMD pad as test Point, diameter 1.0mm")
 		(tags "test point SMD pad")
@@
 	)
 	(gr_rect
-		(start 137.115 101.052746)
-		(end 144.015 102.952747)
+		(start 137.56 103.87)
+		(end 144.46 105.770001)
 		(stroke
 			(width 0.1)
@@
 	)
 	(via
-		(at 143.475 104.45)
+		(at 143.92 107.267254)
 		(size 0.6)
 		(drill 0.3)
@@
 	)
 	(via
-		(at 147.195 108.15)
+		(at 147.64 110.967254)
 		(size 0.6)
 		(drill 0.3)
@@
 	)
 	(via
-		(at 147.195 105.63)
+		(at 147.64 108.447254)
 		(size 0.6)
 		(drill 0.3)
@@
 	)
 	(via
-		(at 143.475 101.81)
+		(at 143.92 104.627254)
 		(size 0.6)
 		(drill 0.3)
@@
 	)
 	(via
-		(at 143.475 103.08)
+		(at 143.92 105.897254)
 		(size 0.6)
 		(drill 0.3)
@@
 	)
 	(via
-		(at 147.195 106.94)
+		(at 147.64 109.757254)
 		(size 0.6)
 		(drill 0.3)
@@
 	)
 	(via
-		(at 147.495 100.442747)
+		(at 147.94 103.260001)
 		(size 0.6)
 		(drill 0.3)
@@
 	)
 	(via
-		(at 143.475 109.55)
+		(at 143.92 112.367254)
 		(size 0.6)
 		(drill 0.3)
@@
 	)
 	(via
-		(at 143.475 108.27)
+		(at 143.92 111.087254)
 		(size 0.6)
 		(drill 0.3)
@@
 	)
 	(via
-		(at 143.475 105.66)
+		(at 143.92 108.477254)
 		(size 0.6)
 		(drill 0.3)
@@
 	)
 	(via
-		(at 147.195 109.47)
+		(at 147.64 112.287254)
 		(size 0.6)
 		(drill 0.3)
@@
 	)
 	(via
-		(at 143.475 106.97)
+		(at 143.92 109.787254)
 		(size 0.6)
 		(drill 0.3)
@@
 	)
 	(via
-		(at 143.475 100.56)
+		(at 143.92 103.377254)
 		(size 0.6)
 		(drill 0.3)
@@
 	)
 	(via
-		(at 132.715 104.952747)
+		(at 133.16 107.770001)
 		(size 0.6)
 		(drill 0.3)
@@
 	)
 	(via
-		(at 132.325 100.502747)
+		(at 132.77 103.320001)
 		(size 0.6)
 		(drill 0.3)
@@
 	)
 	(via
-		(at 133.905 106.96)
+		(at 134.35 109.777254)
 		(size 0.6)
 		(drill 0.3)
@@
 	)
 	(via
-		(at 133.895 108.19)
+		(at 134.34 111.007254)
 		(size 0.6)
 		(drill 0.3)
@@
 	)
 	(via
-		(at 131.565 100.492747)
+		(at 132.01 103.310001)
 		(size 0.6)
 		(drill 0.3)
@@
 	)
 	(segment
-		(start 136.93 103.115)
-		(end 135.855 103.115)
+		(start 137.375 105.932254)
+		(end 136.3 105.932254)
 		(width 0.3)
 		(layer "F.Cu")
@@
 	)
 	(segment
-		(start 137.485 102.56)
-		(end 136.93 103.115)
+		(start 137.93 105.377254)
+		(end 137.375 105.932254)
 		(width 0.3)
 		(layer "F.Cu")
@@
 	)
 	(segment
-		(start 137.485 101.14)
-		(end 137.485 102.56)
+		(start 137.93 103.957254)
+		(end 137.93 105.377254)
 		(width 0.3)
 		(layer "F.Cu")
@@
 	)
 	(segment
-		(start 130.737747 103.47)
-		(end 131.755 103.47)
+		(start 131.182747 106.287254)
+		(end 132.2 106.287254)
 		(width 0.6)
 		(layer "F.Cu")
@@
 	)
 	(segment
-		(start 135.855 100.575)
-		(end 136.92 100.575)
+		(start 136.3 103.392254)
+		(end 137.365 103.392254)
 		(width 0.3)
 		(layer "F.Cu")
@@
 	)
 	(segment
-		(start 136.92 100.575)
-		(end 137.485 101.14)
+		(start 137.365 103.392254)
+		(end 137.93 103.957254)
 		(width 0.3)
 		(layer "F.Cu")
@@
 	)
 	(segment
-		(start 146.202747 104.385)
-		(end 147.495 103.092747)
+		(start 146.647747 107.202254)
+		(end 147.94 105.910001)
 		(width 0.6)
 		(layer "F.Cu")
@@
 	)
 	(segment
-		(start 145.305 104.385)
-		(end 146.202747 104.385)
+		(start 145.75 107.202254)
+		(end 146.647747 107.202254)
 		(width 0.6)
 		(layer "F.Cu")
@@
 	)
 	(segment
-		(start 147.495 103.092747)
-		(end 149.42 103.092747)
+		(start 147.94 105.910001)
+		(end 149.865 105.910001)
 		(width 0.6)
 		(layer "F.Cu")
@@
 	)
 	(segment
-		(start 145.305 103.115)
-		(end 147.472747 103.115)
+		(start 145.75 105.932254)
+		(end 147.917747 105.932254)
 		(width 0.6)
 		(layer "F.Cu")
@@
 	)
 	(segment
-		(start 147.472747 103.115)
-		(end 147.495 103.092747)
+		(start 147.917747 105.932254)
+		(end 147.94 105.910001)
 		(width 0.6)
 		(layer "F.Cu")
@@
 		(polygon
 			(pts
-				(xy 142.975 99.97) (xy 150.525 99.97) (xy 150.52 101.767747) (xy 147.728392 104.767686) (xy 147.705 110.08)
-				(xy 142.975 110.070307)
+				(xy 143.42 102.787254) (xy 150.97 102.787254) (xy 150.965 104.585001) (xy 148.173392 107.58494)
+				(xy 148.15 112.897254) (xy 143.42 112.887561)
 			)
 		)
@@
 		(polygon
 			(pts
-				(xy 130.791506 102.611579) (xy 137.03 102.617099) (xy 137.03 103.695) (xy 134.605 103.695) (xy 132.742217 104.211095)
-				(xy 130.778485 104.194949)
+				(xy 131.236506 105.428833) (xy 137.475 105.434353) (xy 137.475 106.512254) (xy 135.05 106.512254)
+				(xy 133.187217 107.028349) (xy 131.223485 107.012203)
 			)
 		)
@@
 		(polygon
 			(pts
-				(xy 134.547494 101.288524) (xy 137.025 101.29) (xy 137.025 110.139739) (xy 134.465 110.14) (xy 130.778485 104.194949)
-				(xy 130.77646 100.09862) (xy 132.811476 100.097614)
+				(xy 134.992494 104.105778) (xy 137.47 104.107254) (xy 137.47 112.956993) (xy 134.91 112.957254)
+				(xy 131.223485 107.012203) (xy 131.22146 102.915874) (xy 133.256476 102.914868)
 			)
 		)
