File: hardware/Stuttgart.kicad_pcb (KiCad board)
At the start: 2 copper layers, 94.7 x 54 mm, 78 parts, among them IC1 NCV1117ST33T3G, IC2 UCC33420QRAQRQ1, IC3 ISOUSB111DWR, IC6 MCP3202-CI_SN, IC7 MCP251863T-E_9PX, J1 USB_C_Receptacle_USB2.0_16P, J2 FCR7350B, J3 FCR7350G, J4 FCR7350Y, J5 SM03B-SRSS-TB_LF__SN_, U1 RP2354A, U2 TPD2EUSB30, Y1 ABM8-272-T3, Y2 Crystal_GND24

Commit message: Schematic and PCB layout near final
Parts:
- moved C11 31.2 mm to (98.3, 91.1), turned to 180 degrees
- moved IC2 30.6 mm to (89.2, 91.8)
- moved TP6 30.6 mm to (97.1, 93.4)
- moved C20 30.6 mm to (93.5, 92.5)
- moved C21 30.6 mm to (95.1, 92.5)
- moved C19 30.5 mm to (85.3, 91.2)
- moved C18 30.5 mm to (83.8, 91.2)
- moved R12 29.8 mm to (86.3, 88.7), turned to 180 degrees
- moved C12 20.5 mm to (111.2, 88.1)
- moved IC1 19.5 mm to (104.7, 88.8)
- moved TP1 17.3 mm to (110.1, 91.1)
- moved J5 16.1 mm to (121.7, 86.2), turned to 0 degrees
- moved R2 12.5 mm to (111.2, 64.8), turned to 0 degrees
- moved FB1 11.3 mm to (83.5, 87.8), turned to -90 degrees
- moved TP2 11.2 mm to (113.6, 64.5)
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Connections:
- C11 pad 1: VBUS -> +5V
- C11 pad 2: GND -> GND1
- C12 pad 2: GND -> GND1
- C28 pad 1: +3.3VA -> +3V3
- C29 pad 1: +3.3VA -> +3V3
- C30 pad 1: +3.3VA -> +3V3
- C31 pad 1: +3.3VA -> +3V3
- IC1 pad 1: GND -> GND1
- IC1 pad 3: VBUS -> +5V
- IC6 pad 1: SPI1_CS_ISO -> SPI1_CS
- IC6 pad 5: SPI1_TX_ISO -> SPI1_TX
- IC6 pad 6: SPI1_RX_ISO -> SPI1_RX
- IC6 pad 7: SPI1_SCK_ISO -> SPI1_SCK
- IC6 pad 8: +3.3VA -> +3V3
- IC7 pad 14: +3.3VA -> +3V3
- IC7 pad 22: SPI0_SCK_ISO -> SPI0_SCK
- IC7 pad 23: SPI0_TX_ISO -> SPI0_TX
- IC7 pad 24: SPI0_RX_ISO -> SPI0_RX
- IC7 pad 25: SPI0_CS_ISO -> SPI0_CS
- IC7 pad 26: +3.3VA -> +3V3
- IC7 pad 3: CAN_INT_ISO -> CAN_INT
- IC7 pad 8: CAN_INT1_ISO -> CAN_INT1
Routing:
- net +3V3: track 97.6 -> 142.0 mm, vias 4 -> 8
- net +3.3VA: track 26.7 -> 0.00 mm, vias 5 -> 0
- net +5V: track 6.25 -> 32.2 mm, vias 0 -> 2
- net /RP2354A/SWD: track 30.2 -> 12.0 mm, vias 2 -> 0
- net /RP2354A/SWCLK: track 29.0 -> 11.3 mm, vias 3 -> 0
- net +1V1: track 21.4 -> 38.7 mm
- net CAN_INT1: track 9.46 -> 23.2 mm, vias 1 -> 2
- net SPI0_RX: track 5.30 -> 18.6 mm, vias 0 -> 2
- net CAN_INT1_ISO: track 12.1 -> 0.00 mm, vias 2 -> 0
- net SPI1_CS_ISO: track 11.7 -> 0.00 mm
- net USB_D+: track 18.7 -> 30.2 mm, vias 1 -> 0
- net /USB Isolation/VBUS_IN: track 11.0 -> 0.04 mm, vias 2 -> 0
- net GND1: track 68.1 -> 58.3 mm, vias 26 -> 40
- net CAN_INT: track 9.67 -> 19.2 mm, vias 1 -> 2
- net USB_D-: track 20.9 -> 30.2 mm, vias 1 -> 0
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- added copper zone on F.Cu, net /USB Isolation/VBUS_IN
Other:
- board text removed: "SPI0"
- board text removed: "SPI1"

Commit message: Hardware layout complete
Parts:
- moved D3 13.8 mm to (144.8, 70.7)
- moved D4 13.8 mm to (144.8, 90.4)
- moved H1 13.8 mm to (153.3, 90.4)
- moved H2 13.8 mm to (153.3, 70.7)
- moved J2 13.8 mm to (145.1, 100.3)
- moved J3 13.8 mm to (145.1, 80.6)
- moved J4 13.8 mm to (145.1, 60.8)
- moved TP5 12.3 mm to (139.8, 70.7)
- moved TP4 12.2 mm to (139.8, 90.4)
- moved H4 1.53 mm to (108.5, 103.2)
- moved H3 1.30 mm to (108.5, 57.9)
- moved C32 0.36 mm to (133.2, 86.9)
- moved TP6 0.09 mm to (97.1, 93.3)
Connections:
- IC3 pad 6: USB_D- -> /USB Isolation/USB_C_D-
- IC3 pad 7: USB_D+ -> /USB Isolation/USB_C_D+
- J1 pad A6: USB_D+ -> /USB Isolation/USB_C_D+
- J1 pad A7: USB_D- -> /USB Isolation/USB_C_D-
- J1 pad B6: USB_D+ -> /USB Isolation/USB_C_D+
- J1 pad B7: USB_D- -> /USB Isolation/USB_C_D-
- U2 pad 1: USB_D+ -> /USB Isolation/USB_C_D+
- U2 pad 2: USB_D- -> /USB Isolation/USB_C_D-
Routing:
- net +5V: track 32.2 -> 73.6 mm
- net /Vehicle Interface/CAN_L: track 5.79 -> 37.0 mm, vias 0 -> 2
- net /Vehicle Interface/CAN_H: track 5.41 -> 30.4 mm
- net /USB Isolation/USB_C_D-: track 0.00 -> 10.3 mm
- net /USB Isolation/USB_C_D+: track 0.00 -> 9.87 mm
- net USB_D-: track 30.2 -> 20.7 mm
- net USB_D+: track 30.2 -> 20.7 mm
- net GND1: track 58.3 -> 63.8 mm, vias 40 -> 54
- net +3V3: track 142.0 -> 146.4 mm, vias 8 -> 9
- net GND: track 42.1 -> 43.3 mm, vias 6 -> 7
Other:
- board size 94.7 x 54 mm -> 81 x 54 mm
- board text added: "3V3"
- board text added: "ADC"
- board text added: "BLACK"
- board text added: "BLUE"
- board text added: "CAN-H"
- board text added: "CAN-L"
- board text added: "CCU"
- board text added: "DEBUG"
- board text added: "GND"
- board text added: "GREEN"
- board text added: "USB ISO"

Commit message: Board outline and fiducials
Parts:
- added FID1: Fiducial, Fiducial:Fiducial_1mm_Mask2mm, F.Cu at (90.7, 58.0)
- added FID2: Fiducial, Fiducial:Fiducial_1mm_Mask2mm, F.Cu at (154.8, 58.0)
- added FID3: Fiducial, Fiducial:Fiducial_1mm_Mask2mm, F.Cu at (154.7, 103.0)
- added FID4: Fiducial, Fiducial:Fiducial_1mm_Mask2mm, F.Cu at (107.5, 79.5)
- added FID5: Fiducial, Fiducial:Fiducial_1mm_Mask2mm, F.Cu at (121.3, 64.5)
- J4: value FCR7350Y -> FCR7350BL
- moved H3 27.9 mm to (82.8, 68.7)
- moved H4 11.3 mm to (97.2, 102.8)
Other:
- outline, holes or cut-outs redrawn
- board text added: "ISOLATED"
- board text added: "VEHICLE"
- board text removed: "DC-DC"
- board text removed: "USB ISO"
