File: hardware/rp2354a.kicad_sch (KiCad schematic)
At the start: 27 parts, among them J5 SM03B-SRSS-TB_LF__SN_, U1 RP2354A, Y1 ABM8-272-T3

Commit message: Moved GND points, revised DCDC and base USB Work
Connections:
- net GND renamed GND1

Commit message: Schematic Clean Up
Parts:
- J5: JLC Part Number (none) -> C160403
- L1: JLC Part Number (none) -> C42411119
- S1: JLC Part Number (none) -> C5504987
- TP1, TP2: now left out of the parts list
- U1: JLC Part Number (none) -> C41378174
- Y1: JLC Part Number (none) -> C20625731
Connections:
- no-connect marks 0 -> 25
